File: PCB/SnakeHome.kicad_pcb (KiCad board)
At the start: 2 copper layers, 51.5 x 53.5 mm, 31 parts, among them J1 Raspberry_Pi_4, J2 Conn_01x04_Pin, J3 Conn_01x04_Pin, J4 Conn_01x04_Pin, J5 Conn_01x04_Pin, U1 Temp&Humidity_R1, U2 PIR_motion_Kitchen, U3 TCA9548APWR, U4 PIR_motion_Toilet, U5 Temp&Humidity_R2, U6 Temp&Humidity_R3, U7 Temp&Humidity_Kitchen

Commit message: Added RGB Connector
Parts:
- added D1: RGB, Connector_JST:JST_XH_B3B-XH-A_1x03_P2.50mm_Vertical, F.Cu at (111.0, 99.5)
Connections:
- J1 pad 22: unconnected-(J1-GPIO25/SDIO_DAT1-Pad22) -> RGB
Routing:
- net RGB: track 0.00 -> 12.8 mm
- net +5V: track 240.3 -> 244.4 mm
