File: PCB/SnakeHome.kicad_sch (KiCad schematic)
At the start: 7 parts, among them J1 Raspberry_Pi_4, U1 Temp&Humidity_R1, U2 PIR_motion_Kitchen, U4 PIR_motion_Toilet, U5 Temp&Humidity_R2, U6 Temp&Humidity_R3, U7 Temp&Humidity_Kitchen

Commit message: Finished adding the I2C multiplexer to the schem and changing the connectors
Parts:
- added J2, J3, J4, J5: Conn_01x04_Pin, Connector_JST:JST_XH_B4B-XH-A_1x04_P2.50mm_Vertical, symbol Connector:Conn_01x04_Pin
- added R1, R10, R11, R12, R13, R14, R15, R16, R17, R2, R3, R4, R5, R6, R7, R8, R9: R, Resistor_THT:R_Axial_DIN0309_L9.0mm_D3.2mm_P12.70mm_Horizontal, symbol Device:R
- added U3: TCA9548APWR, Package_SO:TSSOP-24_4.4x7.8mm_P0.65mm, symbol Interface_Expansion:TCA9548APWR
- U1, U5, U6, U7: footprint Connector_PinHeader_2.54mm:PinHeader_1x04_P2.54mm_Vertical -> Connector_JST:JST_XH_B4B-XH-A_1x04_P2.50mm_Vertical
- U2, U4: footprint Connector_PinHeader_2.54mm:PinHeader_1x03_P2.54mm_Vertical -> Connector_JST:JST_XH_B3B-XH-A_1x03_P2.50mm_Vertical
Connections:
- net +5V: now also J2.2 (Pin_2), J3.2 (Pin_2), J4.2 (Pin_2), J5.2 (Pin_2), R1.1, R10.1, R11.1, R12.1, R13.1, R14.1, R15.1, R16.1, R17.1, R2.1, R3.1, R4.1, R5.1, R6.1, R7.1, R8.1, R9.1, U3.24 (VCC)
- net GND: now also J2.1 (Pin_1), J3.1 (Pin_1), J4.1 (Pin_1), J5.1 (Pin_1), U3.1 (A0), U3.12 (GND), U3.2 (A1), U3.21 (A2)
- removed net SCL_temp: J1.5 (SCL_I2C1/GPIO03), U1.4 (SCL), U5.4 (SCL), U6.4 (SCL), U7.4 (SCL)
- removed net SDA_temp: J1.3 (SDA_I2C1/GPIO02), U1.2 (SDA), U5.2 (SDA), U6.2 (SDA), U7.2 (SDA)
- new net: R1.2, U3.3 (~{RESET})
- new net SCL_1: J2.3 (Pin_3), R12.2, U3.13 (SD4)
- new net SCL_2: J3.3 (Pin_3), R16.2, U3.15 (SD5)
- new net SCL_3: J4.3 (Pin_3), R13.2, U3.17 (SD6)
- new net SCL_4: J5.3 (Pin_3), R17.2, U3.19 (SD7)
- new net SCL_Bus: J1.5 (SCL_I2C1/GPIO03), U3.22 (SCL)
- new net SCL_Ki: R9.2, U3.10 (SD3), U7.4 (SCL)
- new net SCL_R1: R3.2, U1.4 (SCL), U3.4 (SD0)
- new net SCL_R2: R5.2, U3.6 (SD1), U5.4 (SCL)
- new net SCL_R3: R7.2, U3.8 (SD2), U6.4 (SCL)
- new net SDA_1: J2.4 (Pin_4), R10.2, U3.14 (SC4)
- new net SDA_2: J3.4 (Pin_4), R14.2, U3.16 (SC5)
- new net SDA_3: J4.4 (Pin_4), R11.2, U3.18 (SC6)
- new net SDA_4: J5.4 (Pin_4), R15.2, U3.20 (SC7)
- new net SDA_Bus: J1.3 (SDA_I2C1/GPIO02), U3.23 (SDA)
- new net SDA_Ki: R8.2, U3.11 (SC3), U7.2 (SDA)
- new net SDA_R1: R2.2, U1.2 (SDA), U3.5 (SC0)
- new net SDA_R2: R4.2, U3.7 (SC1), U5.2 (SDA)
- new net SDA_R3: R6.2, U3.9 (SC2), U6.2 (SDA)
Other:
- added sheet I2C_Multiplexer (I2C_Multiplexer.kicad_sch)

Commit message: choosed smd Rs and placed the components on the PCB
Parts:
- added R18, R19: R, Resistor_SMD:R_0402_1005Metric_Pad0.72x0.64mm_HandSolder, symbol Device:R
- R1, R10, R11, R12, R13, R14, R15, R16, R17, R2, R3, R4, R5, R6, R7, R8, R9: footprint Resistor_THT:R_Axial_DIN0309_L9.0mm_D3.2mm_P12.70mm_Horizontal -> Resistor_SMD:R_0402_1005Metric_Pad0.72x0.64mm_HandSolder
Connections:
- net +5V: now also R18.1, R19.1
- net SCL_Bus: now also R18.2
- net SDA_Bus: now also R19.2

Commit message: Added RGB Connector
Parts:
- added D1: SK6812MINI-E, Connector_JST:JST_XH_B3B-XH-A_1x03_P2.50mm_Vertical, symbol neopixel:SK6812MINI-E
Connections:
- net +5V: now also D1.1 (VDD)
- net GND: now also D1.3 (VSS)
- net RGB: now reaches J1.22 (GPIO25/SDIO_DAT1)
- net RGB: now also D1.2 (DIN)
- no-connect marks 0 -> 1
Other:
- sheet Sensors renamed Sensors & RGB
- moved on the sheet: U1, U2, U4, U5, U6, U7
